File: exoMainPCB/exoMainPCB.kicad_sch (KiCad schematic)
At the start: 92 parts, among them J1 Conn_02x06_Odd_Even, J10 Conn_01x03_Pin, J11 USB_A, J12 USB_A, J13 USB_A, J14 Screw_Terminal_01x02, J15 Conn_01x03, J16 Conn_01x02, J17 Screw_Terminal_01x02, J2 HDMI_A, J3 USB_A, J4 Conn_01x02, J5 Conn_01x03, J6 Conn_01x03_Pin, J7 Conn_01x02, J8 Screw_Terminal_01x02, J9 Conn_01x12, SW1 SW_SPDT, SW2 SW_Push, SW3 SW_SPDT, U1 MCP2515-I/ST, U14 SI8642ED-B-IS, U15 SN65HVD230D, U17 SM24CANB-02HTG, U2 MCP2515-I/ST, U3 BNO085, U4 SL2.1A, U5 MCP3008, U7 SN65HVD230D, U8 SM24CANB-02HTG, Y1 16 MHz, Y2 16 MHz, Y3 12 MHz, Y4 32.768 kHz

Commit message: added CAN, HDMI, USB test points, fixed JST connector orientations
Parts:
- added TP1, TP10, TP11, TP12, TP13, TP14, TP15, TP16, TP17, TP18, TP19, TP2, TP20, TP21, TP22, TP23, TP24, TP25, TP26, TP27, TP28, TP29, TP3, TP30, TP4, TP5, TP6, TP7, TP8, TP9: TestPoint, TestPoint:TestPoint_Pad_D1.5mm, symbol Connector:TestPoint
- J10, J6: footprint Connector_PinHeader_2.54mm:PinHeader_1x03_P2.54mm_Vertical -> Connector_JST:JST_GH_BM03B-GHS-TBT_1x03-1MP_P1.25mm_Vertical
- J14, J17, J8: footprint BNO085:1x2 Screw Terminal C3703 -> XT60:CONN-TH_XT60
- J15, J5: footprint Connector_PinSocket_2.54mm:PinSocket_1x03_P2.54mm_Vertical -> Connector_JST:JST_GH_BM03B-GHS-TBT_1x03-1MP_P1.25mm_Vertical
- J16, J4, J7: footprint Connector_PinSocket_2.54mm:PinSocket_1x02_P2.54mm_Vertical -> Connector_JST:JST_GH_BM02B-GHS-TBT_1x02-1MP_P1.25mm_Vertical
Connections:
- net +3V3_{CAN}: now also TP11.1, TP12.1, TP21.1, TP22.1, TP23.1, TP24.1
- net +5V: now also TP4.1, TP5.1, TP6.1, TP7.1, TP8.1, TP9.1
- net D_{CS0}: now also TP16.1
- net D_{CS1}: now also TP13.1
- net D_{HDMI0_HOTPLUG}: now also TP1.1
- net D_{INT0}: now also TP20.1
- net D_{INT1}: now also TP17.1
- net D_{USB_N}: now also TP30.1
- net D_{USB_P}: now also TP29.1
- net GND: now also TP10.1, TP25.1, TP26.1, TP27.1, TP28.1, TP3.1
- net MISO: now also TP14.1, TP18.1
- net MOSI: now also TP15.1, TP19.1
- net at C17.2, U4.16 (XIN), Y3.1: now also TP2.1
Other:
- moved on the sheet: C18, C20, C21, C22, C5, C6, C8, JP1, JP2, JP7, JP8, U14

Commit message: fixed pours and added testpoints to last systems
Parts:
- added TP31, TP32, TP33, TP34, TP35, TP36, TP37, TP38, TP39, TP40, TP41: TestPoint, TestPoint:TestPoint_Pad_D1.5mm, symbol Connector:TestPoint
Connections:
- net IMU_{BOOT}: now also TP37.1
- net IMU_{HINT}: now also TP36.1
- net IMU_{RST}: now also TP38.1
- net P_{IN,+}: now also TP34.1
- net P_{IN,-}: now also TP33.1
- net SG_{IN,+}: now also TP32.1
- net SG_{IN,-}: now also TP31.1
- net V_{battery}: now also TP35.1
- net at JP9.1 (A), Module1.78 (GPIO_VREF(1.8v/3.3v_Input)), Module1.84 (+3.3v_(Output))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: now also TP41.1
- net at C11.1, U3.26 (XOUT32/CLKSEL1), Y4.1: now also TP40.1
- net at C12.1, U3.27 (XIN32), Y4.2: now also TP39.1
Other:
- note added: "Testpoints"
